File: pcb/mcu.kicad_sch (KiCad schematic)
At the start: 12 parts, among them J3 DNP, SW2 SKRKAEE020, SW3 SKRKAEE020, U6 ESP32-S3-WROOM-1

Commit message: Implement RTC and device sync + updated 3d objects
Connections:
- net VBUS_DETECT: now reaches U6.39 (GPIO1/TOUCH1/ADC1_CH0)
- no-connect marks 20 -> 19
Changed lines of the file:
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@@
   (no_connect (at 63.5 78.74))
   (no_connect (at 63.5 88.9))
-  (no_connect (at 154.94 88.9))
   (no_connect (at 63.5 137.16))
   (no_connect (at 154.94 121.92))
@@
     (stroke (width 0) (type default))
   )
-  (wire (pts (xy 26.67 24.13) (xy 36.83 24.13))
+  (wire (pts (xy 30.48 24.13) (xy 45.72 24.13))
     (stroke (width 0) (type default))
   )
@@
     (stroke (width 0) (type default))
   )
+  (wire (pts (xy 30.48 29.21) (xy 45.72 29.21))
+    (stroke (width 0) (type default))
+  )
+  (wire (pts (xy 30.48 19.05) (xy 45.72 19.05))
+    (stroke (width 0) (type default))
+  )
   (wire (pts (xy 259.08 46.99) (xy 241.3 46.99))
     (stroke (width 0) (type default))
@@
     (stroke (width 0) (type default))
   )
-  (wire (pts (xy 36.83 21.59) (xy 26.67 21.59))
+  (wire (pts (xy 30.48 21.59) (xy 45.72 21.59))
     (stroke (width 0) (type default))
   )
@@
     (stroke (width 0) (type default))
   )
+  (wire (pts (xy 30.48 34.29) (xy 45.72 34.29))
+    (stroke (width 0) (type default))
+  )
   (wire (pts (xy 101.6 152.4) (xy 101.6 154.94))
     (stroke (width 0) (type default))
@@
     (stroke (width 0) (type default))
   )
-  (wire (pts (xy 26.67 31.75) (xy 36.83 31.75))
+  (wire (pts (xy 30.48 31.75) (xy 45.72 31.75))
     (stroke (width 0) (type default))
   )
@@
     (stroke (width 0) (type default))
   )
-  (wire (pts (xy 26.67 29.21) (xy 36.83 29.21))
-    (stroke (width 0) (type default))
-  )
-  (wire (pts (xy 36.83 19.05) (xy 26.67 19.05))
-    (stroke (width 0) (type default))
-  )
   (wire (pts (xy 154.94 132.08) (xy 168.91 132.08))
     (stroke (width 0) (type default))
@@
     (stroke (width 0) (type default))
   )
+  (wire (pts (xy 154.94 88.9) (xy 168.91 88.9))
+    (stroke (width 0) (type default))
+  )
   (wire (pts (xy 222.25 90.17) (xy 228.6 90.17))
     (stroke (width 0) (type default))
@@
     (stroke (width 0) (type default))
   )
-  (wire (pts (xy 26.67 26.67) (xy 36.83 26.67))
-    (stroke (width 0) (type default))
-  )
   (wire (pts (xy 109.22 154.94) (xy 109.22 157.48))
     (stroke (width 0) (type default))
@@
     (stroke (width 0) (type default))
   )
+  (wire (pts (xy 30.48 26.67) (xy 45.72 26.67))
+    (stroke (width 0) (type default))
+  )
   (wire (pts (xy 154.94 73.66) (xy 168.91 73.66))
     (stroke (width 0) (type default))
@@
     (effects (font (size 1.27 1.27)) (justify right bottom))
   )
-  (label "~{RTC_INT}" (at 36.83 26.67 180) (fields_autoplaced)
+  (label "~{RTC_INT}" (at 45.72 26.67 180) (fields_autoplaced)
     (effects (font (size 1.27 1.27)) (justify right bottom))
   )
@@
     (effects (font (size 1.27 1.27)) (justify right bottom))
   )
+  (label "VBUS_DETECT" (at 168.91 88.9 180) (fields_autoplaced)
+    (effects (font (size 1.27 1.27)) (justify right bottom))
+  )
   (label "LED_RED" (at 168.91 99.06 180) (fields_autoplaced)
     (effects (font (size 1.27 1.27)) (justify right bottom))
@@
     (effects (font (size 1.27 1.27)) (justify right bottom))
   )
-  (label "DPS_INT" (at 36.83 24.13 180) (fields_autoplaced)
+  (label "DPS_INT" (at 45.72 24.13 180) (fields_autoplaced)
     (effects (font (size 1.27 1.27)) (justify right bottom))
   )
@@
     (effects (font (size 1.27 1.27)) (justify left bottom))
   )
-  (label "USB_D+" (at 36.83 19.05 180) (fields_autoplaced)
-    (effects (font (size 1.27 1.27)) (justify right bottom))
-  )
-  (label "SDA" (at 36.83 31.75 180) (fields_autoplaced)
-    (effects (font (size 1.27 1.27)) (justify right bottom))
-  )
-  (label "SCK" (at 36.83 29.21 180) (fields_autoplaced)
+  (label "USB_D+" (at 45.72 19.05 180) (fields_autoplaced)
+    (effects (font (size 1.27 1.27)) (justify right bottom))
+  )
+  (label "SDA" (at 45.72 31.75 180) (fields_autoplaced)
+    (effects (font (size 1.27 1.27)) (justify right bottom))
+  )
+  (label "SCK" (at 45.72 29.21 180) (fields_autoplaced)
     (effects (font (size 1.27 1.27)) (justify right bottom))
   )
@@
     (effects (font (size 1.27 1.27)) (justify right bottom))
   )
-  (label "USB_D-" (at 36.83 21.59 180) (fields_autoplaced)
+  (label "VBUS_DETECT" (at 45.72 34.29 180) (fields_autoplaced)
+    (effects (font (size 1.27 1.27)) (justify right bottom))
+  )
+  (label "USB_D-" (at 45.72 21.59 180) (fields_autoplaced)
     (effects (font (size 1.27 1.27)) (justify right bottom))
   )
@@
     (effects (font (size 1.27 1.27)) (justify left bottom))
   )
-  (hierarchical_label "SDA" (shape input) (at 26.67 31.75 180) (fields_autoplaced)
-    (effects (font (size 1.27 1.27)) (justify right))
-  )
-  (hierarchical_label "SCK" (shape input) (at 26.67 29.21 180) (fields_autoplaced)
-    (effects (font (size 1.27 1.27)) (justify right))
-  )
-  (hierarchical_label "~{RTC_INT}" (shape input) (at 26.67 26.67 180) (fields_autoplaced)
-    (effects (font (size 1.27 1.27)) (justify right))
-  )
-  (hierarchical_label "USB_D-" (shape input) (at 26.67 21.59 180) (fields_autoplaced)
-    (effects (font (size 1.27 1.27)) (justify right))
-  )
-  (hierarchical_label "DPS_INT" (shape input) (at 26.67 24.13 180) (fields_autoplaced)
-    (effects (font (size 1.27 1.27)) (justify right))
-  )
-  (hierarchical_label "USB_D+" (shape input) (at 26.67 19.05 180) (fields_autoplaced)
-    (effects (font (size 1.27 1.27)) (justify right))
-  )
+  (hierarchical_label "VBUS_DETECT" (shape input) (at 30.48 34.29 180) (fields_autoplaced)
+    (effects (font (size 1.27 1.27)) (justify right))
+  )
+  (hierarchical_label "SDA" (shape input) (at 30.48 31.75 180) (fields_autoplaced)
+    (effects (font (size 1.27 1.27)) (justify right))
+  )
+  (hierarchical_label "SCK" (shape input) (at 30.48 29.21 180) (fields_autoplaced)
+    (effects (font (size 1.27 1.27)) (justify right))
+  )
+  (hierarchical_label "~{RTC_INT}" (shape input) (at 30.48 26.67 180) (fields_autoplaced)
+    (effects (font (size 1.27 1.27)) (justify right))
+  )
+  (hierarchical_label "USB_D-" (shape input) (at 30.48 21.59 180) (fields_autoplaced)
+    (effects (font (size 1.27 1.27)) (justify right))
+  )
+  (hierarchical_label "DPS_INT" (shape input) (at 30.48 24.13 180) (fields_autoplaced)
+    (effects (font (size 1.27 1.27)) (justify right))
+  )
+  (hierarchical_label "USB_D+" (shape input) (at 30.48 19.05 180) (fields_autoplaced)
+    (effects (font (size 1.27 1.27)) (justify right))
+  )
