File: pcb/ot-riwa.kicad_pcb (KiCad board)
At the start: 2 copper layers, 62.9 x 62.5 mm, 63 parts, among them IC1 RV-3028-C7, IC2 DRV5032FB, J1 124018612112A, J2 DNP, J3 DNP, J4 Conn_01x04_Pin, SW1 SKRKAEE020, SW2 SKRKAEE020, SW3 SKRKAEE020, U1 DPS368XTSA1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

Commit message: Refactored components
Parts:
- C13: value 0.1µF -> 0.1uF
- C2, C3: value 10µF -> 10uF
- C4, C5: value 1µF -> 1uF
- U6: value ESP32-S3-WROOM-1 -> ESP32-S3-WROOM-1U-N8
Changed lines of the file:
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@@
         (effects (font (size 1 1) (thickness 0.15)))
     )
-    (fp_text value "ESP32-S3-WROOM-1" (at 0 12) (layer "F.Fab")
+    (fp_text value "ESP32-S3-WROOM-1U-N8" (at 0 12) (layer "F.Fab")
         (effects (font (size 1 1) (thickness 0.15)))
     )
@@
     (property "ki_description" "Mounting Hole with connection")
     (property "ki_keywords" "mounting hole")
-    (attr exclude_from_pos_files)
+    (attr exclude_from_pos_files exclude_from_bom)
     (fp_text reference "H4" (at 0 -3.5 90) (layer "F.SilkS") hide
         (effects (font (size 1 1) (thickness 0.15)))
@@
     (property "ki_description" "Generic connector, single row, 01x02, script generated")
     (property "ki_keywords" "connector")
-    (attr through_hole)
+    (attr through_hole exclude_from_bom)
     (fp_text reference "J2" (at 0 -2.77) (layer "F.SilkS") hide
         (effects (font (size 1 1) (thickness 0.15)))
@@
         (effects (font (size 0.6 0.6) (thickness 0.15)))
     )
-    (fp_text value "0.1µF" (at 0 1.43 90) (layer "F.Fab")
+    (fp_text value "0.1uF" (at 0 1.43 90) (layer "F.Fab")
         (effects (font (size 1 1) (thickness 0.15)))
     )
@@
     (property "ki_description" "Generic connector, single row, 01x04, script generated")
     (property "ki_keywords" "connector")
-    (attr through_hole)
+    (attr through_hole exclude_from_bom)
     (fp_text reference "J4" (at 0 -2.77 90) (layer "F.SilkS") hide
         (effects (font (size 1 1) (thickness 0.15)))
@@
     (pad "2" smd roundrect (at 1 -2.85 180) (size 1 3.5) (layers "F.Cu" "F.Paste" "F.Mask") (roundrect_rratio 0.25)
       (net 19 "GND") (pinfunction "-") (pintype "passive"))
-    (pad "MP" smd roundrect (at -3.35 2.9 180) (size 1.5 3.4) (layers "F.Cu" "F.Paste" "F.Mask") (roundrect_rratio 0.166667))
-    (pad "MP" smd roundrect (at 3.35 2.9 180) (size 1.5 3.4) (layers "F.Cu" "F.Paste" "F.Mask") (roundrect_rratio 0.166667))
+    (pad "MP" smd roundrect (at -3.35 2.9 180) (size 1.5 3.4) (layers "F.Cu" "F.Paste" "F.Mask") (roundrect_rratio 0.1666673333))
+    (pad "MP" smd roundrect (at 3.35 2.9 180) (size 1.5 3.4) (layers "F.Cu" "F.Paste" "F.Mask") (roundrect_rratio 0.1666673333))
     (model "${KIPRJMOD}/components/S2B-PH-SM4-TB--3DModel-STEP-269445.STEP"
       (offset (xyz 0 -4.5 0))
@@
     (property "ki_description" "Mounting Hole with connection")
     (property "ki_keywords" "mounting hole")
-    (attr exclude_from_pos_files)
+    (attr exclude_from_pos_files exclude_from_bom)
     (fp_text reference "H1" (at 0 -3.5 90) (layer "F.SilkS") hide
         (effects (font (size 1 1) (thickness 0.15)))
@@
         (effects (font (size 0.6 0.6) (thickness 0.15)))
     )
-    (fp_text value "10µF" (at 0 1.43 90) (layer "F.Fab")
+    (fp_text value "10uF" (at 0 1.43 90) (layer "F.Fab")
         (effects (font (size 1 1) (thickness 0.15)))
     )
@@
     (property "ki_description" "Mounting Hole with connection")
     (property "ki_keywords" "mounting hole")
-    (attr exclude_from_pos_files)
+    (attr exclude_from_pos_files exclude_from_bom)
     (fp_text reference "H2" (at 0 -3.5 90) (layer "F.SilkS") hide
         (effects (font (size 1 1) (thickness 0.15)))
@@
     (property "ki_description" "Jumper, 2-pole, closed/bridged")
     (property "ki_keywords" "Jumper SPST")
-    (attr exclude_from_pos_files)
+    (attr exclude_from_pos_files exclude_from_bom)
     (net_tie_pad_groups "1, 2")
     (fp_text reference "JP1" (at 0 -1.8 90) (layer "F.SilkS") hide
@@
         (effects (font (size 0.6 0.6) (thickness 0.15)))
     )
-    (fp_text value "1µF" (at 0 1.43) (layer "F.Fab")
+    (fp_text value "1uF" (at 0 1.43) (layer "F.Fab")
         (effects (font (size 1 1) (thickness 0.15)))
     )
@@
     (property "ki_description" "Mounting Hole with connection")
     (property "ki_keywords" "mounting hole")
-    (attr exclude_from_pos_files)
+    (attr exclude_from_pos_files exclude_from_bom)
     (fp_text reference "H3" (at 0 -3.5 90) (layer "F.SilkS") hide
         (effects (font (size 1 1) (thickness 0.15)))
@@
     (property "ki_description" "Generic connector, single row, 01x06, script generated")
     (property "ki_keywords" "connector")
-    (attr through_hole exclude_from_pos_files)
+    (attr through_hole exclude_from_pos_files exclude_from_bom)
     (fp_text reference "J3" (at 0 -2.77 90) (layer "F.SilkS") hide
         (effects (font (size 1 1) (thickness 0.15)))
@@
         (effects (font (size 0.6 0.6) (thickness 0.15)))
     )
-    (fp_text value "1µF" (at 0 1.43) (layer "F.Fab")
+    (fp_text value "1uF" (at 0 1.43) (layer "F.Fab")
         (effects (font (size 1 1) (thickness 0.15)))
     )
@@
         (effects (font (size 0.6 0.6) (thickness 0.15)))
     )
-    (fp_text value "10µF" (at 0 1.43 90) (layer "F.Fab")
+    (fp_text value "10uF" (at 0 1.43 90) (layer "F.Fab")
         (effects (font (size 1 1) (thickness 0.15)))
     )

Commit message: Fixed usage of strapping pins
Parts:
- U6: value ESP32-S3-WROOM-1U-N8 -> ESP32-S3-WROOM-1; footprint ESP32-S3:ESP32-S3-WROOM-1U -> PCM_Espressif:ESP32-S3-WROOM-1U
Connections:
- U6 pad 10: unconnected-(U6-GPIO17/U1TXD/ADC2_CH6-Pad10) -> /main/SCK
- U6 pad 11: unconnected-(U6-GPIO18/U1RXD/ADC2_CH7/CLK_OUT3-Pad11) -> /main/SDA
- U6 pad 15: /main/SCK -> unconnected-(U6-GPIO3/TOUCH3/ADC1_CH2-Pad15)
- U6 pad 16: /main/SDA -> unconnected-(U6-GPIO46-Pad16)
- U6 pad 26: /main/~{RTC_INT} -> unconnected-(U6-GPIO45-Pad26)
- U6 pad 31: unconnected-(U6-GPIO38/FSPIWP/SUBSPIWP-Pad31) -> /main/~{RTC_INT}
Routing:
- net /main/SCK: track 53.3 -> 59.2 mm
- net /main/SDA: track 49.3 -> 54.5 mm
- net /main/~{RTC_INT}: track 26.4 -> 28.2 mm

Commit message: Implement RTC and device sync + updated 3d objects
Parts:
- IC2: moved to B.Cu
- moved TP8 6.08 mm to (108.6, 91.9)
- moved IC2 2.57 mm to (105.6, 96.9), turned to -90 degrees
- moved C13 1.32 mm to (108.5, 96.4), turned to 90 degrees
Routing:
- net /main/PSU/ENABLE: track 35.9 -> 40.8 mm, vias 2 -> 3
- net +BATT: track 36.8 -> 33.3 mm
