File: pcb/rtc.kicad_sch (KiCad schematic)
At the start: 8 parts, among them IC1 RV-3028-C7, SW1 SKRKAEE020

Commit message: Implement RTC and device sync + updated 3d objects
Connections:
- net +3.3V: now also R6.2
- net VBackup: no longer R6.2
Changed lines of the file:
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@@
-    (stroke (width 0) (type default))
-  )
-  (wire (pts (xy 175.26 72.39) (xy 175.26 80.01))
     (stroke (width 0) (type default))
   )
@@
     (stroke (width 0) (type dash))
   )
+  (wire (pts (xy 175.26 76.2) (xy 175.26 80.01))
+    (stroke (width 0) (type default))
+  )
   (wire (pts (xy 113.03 106.68) (xy 113.03 109.22))
     (stroke (width 0) (type default))
@@
     (stroke (width 0) (type default))
   )
-  (wire (pts (xy 175.26 72.39) (xy 185.42 72.39))
-    (stroke (width 0) (type default))
-  )
   (wire (pts (xy 29.21 20.32) (xy 40.64 20.32))
     (stroke (width 0) (type default))
@@
   )
   (label "SCK" (at 40.64 25.4 180) (fields_autoplaced)
-    (effects (font (size 1.27 1.27)) (justify right bottom))
-  )
-  (label "VBackup" (at 185.42 72.39 180) (fields_autoplaced)
     (effects (font (size 1.27 1.27)) (justify right bottom))
   )
@@
         )
       )
+    )
+  )
+  (symbol (lib_id "power:+3.3V") (at 175.26 76.2 0) (unit 1)
+    (in_bom yes) (on_board yes) (dnp no) (fields_autoplaced)
+    (property "Reference" "#PWR030" (at 175.26 80.01 0)
+      (effects (font (size 1.27 1.27)) hide)
+    )
+    (property "Value" "+3.3V" (at 175.26 72.6981 0)
+      (effects (font (size 1.27 1.27)))
+    )
+    (property "Footprint" "" (at 175.26 76.2 0)
+      (effects (font (size 1.27 1.27)) hide)
+    )
+    (property "Datasheet" "" (at 175.26 76.2 0)
+      (effects (font (size 1.27 1.27)) hide)
+    )
+    (pin "1")
+    (instances
+      (project "ot-riwa"
+        (path "/27c79cfd-7e0d-4d78-9eed-2a8b043fdd67/56041fc6-6e17-4b0b-abcc-5d5fefb6b277"
+          (reference "#PWR030") (unit 1)
+        )
+        (path "/27c79cfd-7e0d-4d78-9eed-2a8b043fdd67/56041fc6-6e17-4b0b-abcc-5d5fefb6b277/4e5447bd-0140-4adc-bb38-6eb2d5832537"
+          (reference "#PWR056") (unit 1)
+        )
+      )
+      (project "dps368-breakout"
+        (path "/a87d30f0-0d66-475a-869d-b3a36ef9d8b3"
+          (reference "#PWR010") (unit 1)
+        )
+      )
